File: Bias Current.kicad_sch (KiCad schematic)
At the start: 14 parts, among them Q1 PNP, Q2 PMOS, U1 XTR111AIDGQT, U2 DAC5311IDCKR

Commit message: pcb started
Parts:
- C1: renamed from C2; footprint (none) -> Capacitor_SMD:C_0603_1608Metric_Pad1.08x0.95mm_HandSolder
- C2: renamed from C3; footprint (none) -> Capacitor_SMD:C_0603_1608Metric_Pad1.08x0.95mm_HandSolder
- C3: renamed from C1; footprint (none) -> Capacitor_SMD:C_0603_1608Metric_Pad1.08x0.95mm_HandSolder
- C4: renamed from C9; footprint (none) -> Capacitor_SMD:C_0603_1608Metric_Pad1.08x0.95mm_HandSolder
- JP3: renamed from JP1; footprint (none) -> TestPoint:TestPoint_2Pads_Pitch2.54mm_Drill0.8mm
- Q1: value PNP -> MMBT2907A; footprint (none) -> Package_TO_SOT_SMD:SOT-23
- Q2: value PMOS -> BSP613PH6327XTSA1; footprint (none) -> Package_TO_SOT_SMD:SOT-23
- R10: renamed from R3; footprint (none) -> Resistor_SMD:R_0603_1608Metric_Pad0.98x0.95mm_HandSolder
- R11: renamed from R1; footprint (none) -> Resistor_SMD:R_0603_1608Metric_Pad0.98x0.95mm_HandSolder
- R12: renamed from R4; footprint (none) -> Resistor_SMD:R_0603_1608Metric_Pad0.98x0.95mm_HandSolder
- R13: renamed from R16; footprint (none) -> Resistor_SMD:R_0603_1608Metric_Pad0.98x0.95mm_HandSolder
- R9: renamed from R2; footprint (none) -> Resistor_SMD:R_0603_1608Metric_Pad0.98x0.95mm_HandSolder
- U1: renamed from U2; footprint DCK0006A_N -> Project Footprint Library:DAC5311
- U2: renamed from U1; footprint DGQ0010D_NV_N -> Project Footprint Library:XTR111
Other:
- moved on the sheet: C1, C2, C3, C4, JP3, Q1, Q2, R10, R11, R12, R13, R9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
