File: Fault detection.kicad_sch (KiCad schematic)
At the start: 1 part, among them U10 LP2901D

Commit message: pcb started
Parts:
- removed U10: LP2901D, D14, symbol Project Symbol Library:LP2901D
- added C32: 0.1uF, Capacitor_SMD:C_0603_1608Metric_Pad1.08x0.95mm_HandSolder, symbol Device:C_Small
- added C33, C35: 1000pF, Capacitor_SMD:C_0603_1608Metric_Pad1.08x0.95mm_HandSolder, symbol Device:C_Small
- added C34: 22nF, Capacitor_SMD:C_0603_1608Metric_Pad1.08x0.95mm_HandSolder, symbol Device:C_Small
- added R51: 150K, Resistor_SMD:R_0603_1608Metric_Pad0.98x0.95mm_HandSolder, symbol Device:R_Small_US
- added R52, R54, R55: 100K, Resistor_SMD:R_0603_1608Metric_Pad0.98x0.95mm_HandSolder, symbol Device:R_Small_US
- added R53: 4.99M, Resistor_SMD:R_0603_1608Metric_Pad0.98x0.95mm_HandSolder, symbol Device:R_Small_US
- added R56: 20K, Resistor_SMD:R_0603_1608Metric_Pad0.98x0.95mm_HandSolder, symbol Device:R_Small_US
- added TP6: TestPoint, TestPoint:TestPoint_THTPad_D2.0mm_Drill1.0mm, symbol Connector:TestPoint
- added U8: LP2901D, Package_SO:SOIC-14_3.9x8.7mm_P1.27mm, symbol Comparator:LP2901D
Connections:
- net ACC_OUT: now also R53.1
- net GND: now also C32.2, C33.1, C34.2, C35.1, R56.1, U8.10 (-), U8.11 (+), U8.12 (V-), U8.8 (-), U8.9 (+)
- new net: C34.1, R53.2, TP6.1, U8.4 (-), U8.7 (+)
- new net: C33.2, R51.1, R54.2, U8.5 (+)
- new net: C35.2, R54.1, R56.2, U8.6 (-)
- new net DVDD: R52.2, R55.2
- new net OPEN_ERR: R52.1, U8.2
- new net SHORT_ERR: R55.1, U8.1
- new net VCC_24V: C32.1, R51.2, U8.3 (V+)
Other:
- note added: "detects open circuit and high voltage Input Voltage > 11V"
