File: IEPE Texas Instruments TIDUD62 Receiver.kicad_sch (KiCad schematic)
At the start: 11 parts, among them J1 Conn_Coaxial, J2 Conn_01x20_Pin

Commit message: pcb started
Parts:
- added D3: RED, Diode_SMD:D_0603_1608Metric_Pad1.05x0.95mm_HandSolder, symbol Device:LED
- added JP1, JP2: Jumper_2_Open, TestPoint:TestPoint_2Pads_Pitch2.54mm_Drill0.8mm, symbol Jumper:Jumper_2_Open
- added R8: 820E, Resistor_SMD:R_0603_1608Metric_Pad0.98x0.95mm_HandSolder, symbol Device:R_Small_US
- D1: renamed from D2; footprint (none) -> Diode_SMD:D_0603_1608Metric_Pad1.05x0.95mm_HandSolder
- D2: renamed from D3; footprint (none) -> Diode_SMD:D_0603_1608Metric_Pad1.05x0.95mm_HandSolder
- J1: renamed from J2; footprint (none) -> Connector_PinHeader_2.54mm:PinHeader_1x20_P2.54mm_Vertical
- J2: renamed from J1; footprint (none) -> Connector_Coaxial:BNC_TEConnectivity_1478035_Horizontal
- R1: renamed from R9; footprint (none) -> Resistor_SMD:R_0603_1608Metric_Pad0.98x0.95mm_HandSolder
- R2: renamed from R10; footprint (none) -> Resistor_SMD:R_0603_1608Metric_Pad0.98x0.95mm_HandSolder
- R3: renamed from R11; footprint (none) -> Resistor_SMD:R_0603_1608Metric_Pad0.98x0.95mm_HandSolder
- R4: renamed from R12; footprint (none) -> Resistor_SMD:R_0603_1608Metric_Pad0.98x0.95mm_HandSolder
- R5: renamed from R13; footprint (none) -> Resistor_SMD:R_0603_1608Metric_Pad0.98x0.95mm_HandSolder
- R6: renamed from R51; footprint (none) -> Resistor_SMD:R_0603_1608Metric_Pad0.98x0.95mm_HandSolder
- R7: renamed from R50; footprint (none) -> Resistor_SMD:R_0603_1608Metric_Pad0.98x0.95mm_HandSolder
Connections:
- net Bias Current/ACC_OUT: now also JP1.2 (B); no longer J2.1 (In)
- net DVDD: now also R8.1
- net GND: now also D3.1 (K)
- new net: D3.2 (A), R8.2
- new net DC Bias and Attenueator/ACC_OUT: JP2.1 (A)
- new net Fault detection/ACC_OUT: J2.1 (In), JP1.1 (A), JP2.2 (B)
Other:
- sheet ADC ports: added ADC_CS, DIN, DOUT, DRDY, HR_mode, RESET, SCLK; removed none
- sheet Bias Current ports: added VCC_24V; removed none
- sheet Fault detection ports: added DVDD, OPEN_ERR, SHORT_ERR, VCC_24V; removed none
- sheet SPI_Shift register ports: added DIN, SCLK, SR_CS; removed none
