File: SPI_Shift_register.kicad_sch (KiCad schematic)
At the start: 6 parts, among them J4 Conn_01x10_Pin, J5 SR_EN, U8 SN74HC595PW

Commit message: pcb started
Parts:
- C40: renamed from C32; footprint (none) -> Capacitor_SMD:C_0603_1608Metric_Pad1.08x0.95mm_HandSolder
- J4: footprint (none) -> Connector_PinHeader_2.54mm:PinHeader_1x10_P2.54mm_Vertical
- J5: footprint (none) -> Connector_PinHeader_2.54mm:PinHeader_1x02_P2.54mm_Vertical
- R60: renamed from R48; footprint (none) -> Resistor_SMD:R_0603_1608Metric_Pad0.98x0.95mm_HandSolder
- R61: renamed from R49; footprint (none) -> Resistor_SMD:R_0603_1608Metric_Pad0.98x0.95mm_HandSolder
- U10: renamed from U8; value SN74HC595PW -> SN74HC595PWR; footprint PW16 -> Project Footprint Library:SN74HC595
Connections:
- net CS renamed SR_CS
Changed lines of the file:
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@@
+	(wire
+		(pts
+			(xy 34.29 154.94) (xy 59.69 154.94)
+		)
+		(stroke
+			(width 0)
+			(type default)
+		)
+	)
 	(wire
 		(pts
@@
 	(wire
 		(pts
+			(xy 34.29 151.13) (xy 59.69 151.13)
+		)
+		(stroke
+			(width 0)
+			(type default)
+		)
+	)
+	(wire
+		(pts
 			(xy 181.61 83.82) (xy 200.66 83.82)
 		)
@@
 		(pts
 			(xy 181.61 81.28) (xy 181.61 83.82)
+		)
+		(stroke
+			(width 0)
+			(type default)
+		)
+	)
+	(wire
+		(pts
+			(xy 36.83 146.05) (xy 60.96 146.05)
 		)
 		(stroke
@@
 		)
 	)
-	(label "CS"
+	(label "SR_CS"
 		(at 187.96 93.98 0)
 		(fields_autoplaced yes)
@@
 		)
 	)
+	(label "SCLK"
+		(at 59.69 154.94 0)
+		(fields_autoplaced yes)
+		(effects
+			(font
+				(size 1.27 1.27)
+			)
+			(justify left bottom)
+		)
+	)
 	(label "DVDD"
 		(at 200.66 76.2 0)
@@
 		)
 	)
+	(label "DIN"
+		(at 59.69 151.13 0)
+		(fields_autoplaced yes)
+		(effects
+			(font
+				(size 1.27 1.27)
+			)
+			(justify left bottom)
+		)
+	)
 	(label "RESET"
 		(at 59.69 138.43 0)
+		(fields_autoplaced yes)
+		(effects
+			(font
+				(size 1.27 1.27)
+			)
+			(justify left bottom)
+		)
+	)
+	(label "SR_CS"
+		(at 60.96 146.05 0)
 		(fields_autoplaced yes)
 		(effects
@@
 		)
 	)
+	(hierarchical_label "SCLK"
+		(shape input)
+		(at 34.29 154.94 180)
+		(fields_autoplaced yes)
+		(effects
+			(font
+				(size 1.27 1.27)
+			)
+			(justify right)
+		)
+	)
+	(hierarchical_label "SR_CS"
+		(shape input)
+		(at 36.83 146.05 180)
+		(fields_autoplaced yes)
+		(effects
+			(font
+				(size 1.27 1.27)
+			)
+			(justify right)
+		)
+	)
 	(hierarchical_label "GAIN_SEL1"
 		(shape input)
@@
 		(shape input)
 		(at 34.29 130.81 180)
+		(fields_autoplaced yes)
+		(effects
+			(font
+				(size 1.27 1.27)
+			)
+			(justify right)
+		)
+	)
+	(hierarchical_label "DIN"
+		(shape input)
+		(at 34.29 151.13 180)
 		(fields_autoplaced yes)
 		(effects
@@
 		(on_board yes)
 		(dnp no)
-		(property "Reference" "R48"
+		(property "Reference" "R60"
 			(at 203.2 93.726 90)
 			(effects
@@
 			)
 		)
-		(property "Footprint" ""
+		(property "Footprint" "Resistor_SMD:R_0603_1608Metric_Pad0.98x0.95mm_HandSolder"
 			(at 203.2 91.44 0)
 			(effects
@@
 			(project "IEPE Texas Instruments TIDUD62 Receiver"
 				(path "/b0c16732-dcc2-48d1-93ba-25fcc89f81c2/3a9b049a-9840-4d4c-a2f0-f9a7637055c1"
-					(reference "R48")
+					(reference "R60")
 					(unit 1)
 				)
@@
 			)
 		)
-		(property "Footprint" ""
+		(property "Footprint" "Connector_PinHeader_2.54mm:PinHeader_1x02_P2.54mm_Vertical"
 			(at 219.71 105.41 0)
 			(effects
@@
 		(on_board yes)
 		(dnp no)
-		(property "Reference" "#PWR049"
+		(property "Reference" "#PWR064"
 			(at 181.61 67.31 0)
 			(effects
@@
 			(project "IEPE Texas Instruments TIDUD62 Receiver"
 				(path "/b0c16732-dcc2-48d1-93ba-25fcc89f81c2/3a9b049a-9840-4d4c-a2f0-f9a7637055c1"
-					(reference "#PWR049")
+					(reference "#PWR064")
 					(unit 1)
 				)
@@
 			)
 		)
-		(property "Footprint" ""
+		(property "Footprint" "Connector_PinHeader_2.54mm:PinHeader_1x10_P2.54mm_Vertical"
 			(at 100.33 58.42 0)
 			(effects
@@
 		(on_board yes)
 		(dnp no)
-		(property "Reference" "R49"
+		(property "Reference" "R61"
 			(at 181.61 101.346 90)
 			(effects
@@
 			)
 		)
-		(property "Footprint" ""
+		(property "Footprint" "Resistor_SMD:R_0603_1608Metric_Pad0.98x0.95mm_HandSolder"
 			(at 181.61 99.06 0)
 			(effects
@@
 			(project "IEPE Texas Instruments TIDUD62 Receiver"
 				(path "/b0c16732-dcc2-48d1-93ba-25fcc89f81c2/3a9b049a-9840-4d4c-a2f0-f9a7637055c1"
-					(reference "R49")
+					(reference "R61")
 					(unit 1)
 				)
@@
 		(on_board yes)
 		(dnp no)
-		(property "Reference" "#PWR051"
+		(property "Reference" "#PWR066"
 			(at 214.63 121.92 0)
 			(effects
@@
 			(project "IEPE Texas Instruments TIDUD62 Receiver"
 				(path "/b0c16732-dcc2-48d1-93ba-25fcc89f81c2/3a9b049a-9840-4d4c-a2f0-f9a7637055c1"
-					(reference "#PWR051")
+					(reference "#PWR066")
 					(unit 1)
 				)
@@
 		(on_board yes)
 		(dnp no)
-		(property "Reference" "#PWR048"
+		(property "Reference" "#PWR065"
 			(at 110.49 110.49 0)
 			(effects
@@
 			(project "IEPE Texas Instruments TIDUD62 Receiver"
 				(path "/b0c16732-dcc2-48d1-93ba-25fcc89f81c2/3a9b049a-9840-4d4c-a2f0-f9a7637055c1"
-					(reference "#PWR048")
+					(reference "#PWR065")
 					(unit 1)
 				)
@@
 		(on_board yes)
 		(dnp no)
-		(property "Reference" "#PWR050"
+		(property "Reference" "#PWR063"
 			(at 90.17 72.39 0)
 			(effects
@@
 			(project "IEPE Texas Instruments TIDUD62 Receiver"
 				(path "/b0c16732-dcc2-48d1-93ba-25fcc89f81c2/3a9b049a-9840-4d4c-a2f0-f9a7637055c1"
-					(reference "#PWR050")
+					(reference "#PWR063")
 					(unit 1)
 				)
@@
 		(dnp no)
 		(fields_autoplaced yes)
-		(property "Reference" "U8"
+		(property "Reference" "U10"
 			(at 146.05 73.66 0)
 			(effects
@@
 			)
 		)
-		(property "Value" "SN74HC595PW"
+		(property "Value" "SN74HC595PWR"
 			(at 146.05 76.2 0)
 			(effects
@@
 			)
 		)
-		(property "Footprint" "PW16"
+		(property "Footprint" "Project Footprint Library:SN74HC595"
 			(at 115.57 83.82 0)
 			(effects
@@
 			(project "IEPE Texas Instruments TIDUD62 Receiver"
 				(path "/b0c16732-dcc2-48d1-93ba-25fcc89f81c2/3a9b049a-9840-4d4c-a2f0-f9a7637055c1"
-					(reference "U8")
+					(reference "U10")
 					(unit 1)
 				)
@@
 		(dnp no)
 		(fields_autoplaced yes)
-		(property "Reference" "C32"
+		(property "Reference" "C40"
 			(at 184.15 77.4762 0)
 			(effects
@@
 			)
 		)
-		(property "Footprint" ""
+		(property "Footprint" "Capacitor_SMD:C_0603_1608Metric_Pad1.08x0.95mm_HandSolder"
 			(at 181.61 78.74 0)
 			(effects
@@
 			(project "IEPE Texas Instruments TIDUD62 Receiver"
 				(path "/b0c16732-dcc2-48d1-93ba-25fcc89f81c2/3a9b049a-9840-4d4c-a2f0-f9a7637055c1"
-					(reference "C32")
+					(reference "C40")
 					(unit 1)
 				)
